File: tps63001-slim.kicad_pcb (KiCad board)
At the start: 2 copper layers, 15.7 x 15.7 mm, 10 parts, among them J1 Conn_01x04_Male, U1 TPS63001

Commit message: board routed
Routing:
- net Earth: track 0.00 -> 38.0 mm, vias 0 -> 4
- net Net-(C4-Pad1): track 0.00 -> 33.2 mm, vias 0 -> 1
- net Net-(C1-Pad1): track 0.00 -> 22.5 mm, vias 0 -> 1
- net Net-(L1-Pad1): track 0.00 -> 5.21 mm
- net Net-(L1-Pad2): track 0.00 -> 5.21 mm
- net Net-(J1-Pad1): track 0.00 -> 4.33 mm
Changed lines of the file:
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@@
     (effects (font (size 1 1) (thickness 0.15)) (justify mirror))
   )
+  (segment (start 106.5879 108.0446) (end 106.85 107.7825) (width 0.2502) (layer "F.Cu") (net 1))
+  (segment (start 107.7366 110.6575) (end 107.4257 110.6575) (width 0.5) (layer "F.Cu") (net 1))
+  (segment (start 107.4257 110.6575) (end 107.35 110.6575) (width 0.2502) (layer "F.Cu") (net 1))
+  (segment (start 104.648 108.1825) (end 104.7859 108.0446) (width 0.5) (layer "F.Cu") (net 1))
+  (segment (start 106.104 108.0446) (end 106.5879 108.0446) (width 0.5) (layer "F.Cu") (net 1))
+  (segment (start 111.607 113.8) (end 110.0564 112.2494) (width 0.5) (layer "F.Cu") (net 1))
+  (segment (start 102.616 106.273) (end 102.616 108.1825) (width 0.5) (layer "F.Cu") (net 1))
+  (segment (start 108.7456 112.2494) (end 107.7744 111.2782) (width 0.5) (layer "F.Cu") (net 1))
+  (segment (start 102.616 108.1825) (end 104.648 108.1825) (width 0.5) (layer "F.Cu") (net 1))
+  (segment (start 110.0564 112.2494) (end 108.7456 112.2494) (width 0.5) (layer "F.Cu") (net 1))
+  (segment (start 107.7744 111.2782) (end 107.7744 110.6953) (width 0.5) (layer "F.Cu") (net 1))
+  (segment (start 104.7859 108.0446) (end 106.104 108.0446) (width 0.5) (layer "F.Cu") (net 1))
+  (segment (start 107.85 110.6575) (end 107.8122 110.6953) (width 0.2502) (layer "F.Cu") (net 1))
+  (segment (start 102.108 105.765) (end 102.616 106.273) (width 0.5) (layer "F.Cu") (net 1))
+  (segment (start 107.8122 110.6953) (end 107.7744 110.6953) (width 0.2502) (layer "F.Cu") (net 1))
+  (segment (start 107.7744 110.6953) (end 107.7366 110.6575) (width 0.5) (layer "F.Cu") (net 1))
+  (via (at 106.104 108.0446) (size 0.8) (drill 0.4) (layers "F.Cu" "B.Cu") (net 1))
+  (segment (start 111.607 113.8) (end 111.607 111.019) (width 0.5) (layer "B.Cu") (net 1))
+  (segment (start 111.607 111.019) (end 108.6326 108.0446) (width 0.5) (layer "B.Cu") (net 1))
+  (segment (start 108.6326 108.0446) (end 106.104 108.0446) (width 0.5) (layer "B.Cu") (net 1))
+  (segment (start 114.9178 108.1157) (end 112.776 110.2575) (width 0.5) (layer "F.Cu") (net 2))
+  (segment (start 107.15 109.22) (end 107.85 109.22) (width 0.5) (layer "F.Cu") (net 2))
+  (segment (start 108.35 109.22) (end 108.35 109.7693) (width 0.5) (layer "F.Cu") (net 2))
+  (segment (start 100.4604 104.1626) (end 100.4604 108.1019) (width 0.5) (layer "F.Cu") (net 2))
+  (segment (start 107.85 109.22) (end 107.85 108.6707) (width 0.5) (layer "F.Cu") (net 2))
+  (segment (start 113.284 102.515) (end 114.9178 104.1488) (width 0.5) (layer "F.Cu") (net 2))
+  (segment (start 114.9178 104.1488) (end 114.9178 108.1157) (width 0.5) (layer "F.Cu") (net 2))
+  (segment (start 104.648 110.2575) (end 105.6855 109.22) (width 0.5) (layer "F.Cu") (net 2))
+  (segment (start 107.85 109.22) (end 108.35 109.22) (width 0.5) (layer "F.Cu") (net 2))
+  (segment (start 108.55 109.22) (end 109.7065 109.22) (width 0.5) (layer "F.Cu") (net 2))
+  (segment (start 105.6855 109.22) (end 107.15 109.22) (width 0.5) (layer "F.Cu") (net 2))
+  (segment (start 109.7065 109.22) (end 110.744 110.2575) (width 0.5) (layer "F.Cu") (net 2))
+  (segment (start 108.35 109.7693) (end 108.35 110.6575) (width 0.2502) (layer "F.Cu") (net 2))
+  (segment (start 107.85 108.6707) (end 107.85 107.7825) (width 0.2502) (layer "F.Cu") (net 2))
+  (segment (start 112.776 110.2575) (end 110.744 110.2575) (width 0.5) (layer "F.Cu") (net 2))
+  (segment (start 102.616 110.2575) (end 104.648 110.2575) (width 0.5) (layer "F.Cu") (net 2))
+  (segment (start 108.35 109.22) (end 108.55 109.22) (width 0.5) (layer "F.Cu") (net 2))
+  (segment (start 100.4604 108.1019) (end 102.616 110.2575) (width 0.5) (layer "F.Cu") (net 2))
+  (segment (start 102.108 102.515) (end 100.4604 104.1626) (width 0.5) (layer "F.Cu") (net 2))
+  (via (at 114.808 101.092) (size 0.8) (drill 0.4) (layers "F.Cu" "B.Cu") (free) (net 2))
+  (via (at 101.092 114.808) (size 0.8) (drill 0.4) (layers "F.Cu" "B.Cu") (free) (net 2))
+  (via (at 101.092 101.092) (size 0.8) (drill 0.4) (layers "F.Cu" "B.Cu") (free) (net 2))
+  (via (at 114.808 114.808) (size 0.8) (drill 0.4) (layers "F.Cu" "B.Cu") (free) (net 2))
+  (segment (start 109.067 113.8) (end 109.067 112.4997) (width 0.5) (layer "B.Cu") (net 2))
+  (segment (start 108.55 111.9827) (end 109.067 112.4997) (width 0.5) (layer "B.Cu") (net 2))
+  (segment (start 108.55 109.22) (end 108.55 111.9827) (width 0.5) (layer "B.Cu") (net 2))
+  (segment (start 107.85 109.22) (end 108.55 109.22) (width 0.5) (layer "B.Cu") (net 2))
+  (segment (start 106.225 106.1993) (end 106.3657 106.1993) (width 0.25) (layer "F.Cu") (net 3))
+  (segment (start 107.35 107.1836) (end 107.35 107.7825) (width 0.25) (layer "F.Cu") (net 3))
+  (segment (start 106.225 103.124) (end 106.225 106.1993) (width 0.25) (layer "F.Cu") (net 3))
+  (segment (start 106.3657 106.1993) (end 107.35 107.1836) (width 0.25) (layer "F.Cu") (net 3))
+  (segment (start 103.987 113.8) (end 106.85 110.937) (width 0.25) (layer "F.Cu") (net 4))
+  (segment (start 106.85 110.937) (end 106.85 110.6575) (width 0.25) (layer "F.Cu") (net 4))
+  (segment (start 109.475 103.124) (end 109.475 106.1993) (width 0.25) (layer "F.Cu") (net 5))
+  (segment (start 109.475 106.1993) (end 109.3343 106.1993) (width 0.25) (layer "F.Cu") (net 5))
+  (segment (start 108.35 107.1836) (end 108.35 107.7825) (width 0.25) (layer "F.Cu") (net 5))
+  (segment (start 109.3343 106.1993) (end 108.35 107.1836) (width 0.25) (layer "F.Cu") (net 5))
+  (segment (start 113.284 105.765) (end 113.284 107.6745) (width 0.25) (layer "F.Cu") (net 6))
+  (segment (start 110.344 107.7825) (end 109.5116 107.7825) (width 0.25) (layer "F.Cu") (net 6))
+  (segment (start 110.744 108.1825) (end 110.344 107.7825) (width 0.25) (layer "F.Cu") (net 6))
+  (segment (start 113.284 114.31205) (end 113.284 113.28225) (width 0.25) (layer "F.Cu") (net 6))
+  (segment (start 113.284 113.28225) (end 111.25375 111.252) (width 0.25) (layer "F.Cu") (net 6))
+  (segment (start 109.4445 111.252) (end 108.85 110.6575) (width 0.25) (layer "F.Cu") (net 6))
+  (segment (start 111.25375 111.252) (end 109.4445 111.252) (width 0.25) (layer "F.Cu") (net 6))
+  (segment (start 113.284 107.6745) (end 112.776 108.1825) (width 0.25) (layer "F.Cu") (net 6))
+  (segment (start 112.28005 115.316) (end 113.284 114.31205) (width 0.25) (layer "F.Cu") (net 6))
+  (segment (start 109.5116 107.7825) (end 108.85 107.7825) (width 0.25) (layer "F.Cu") (net 6))
+  (segment (start 110.744 108.1825) (end 112.776 108.1825) (width 0.25) (layer "F.Cu") (net 6))
+  (segment (start 106.527 114.655) (end 107.188 115.316) (width 0.25) (layer "F.Cu") (net 6))
+  (segment (start 106.527 113.8) (end 106.527 114.655) (width 0.25) (layer "F.Cu") (net 6))
+  (segment (start 107.188 115.316) (end 112.28005 115.316) (width 0.25) (layer "F.Cu") (net 6))
+  (segment (start 109.5116 107.0594) (end 109.5116 107.7825) (width 0.25) (layer "F.Cu") (net 6))
+  (via (at 109.5116 107.0594) (size 0.8) (drill 0.4) (layers "F.Cu" "B.Cu") (net 6))
+  (segment (start 106.527 112.6247) (end 105.3764 111.4741) (width 0.25) (layer "B.Cu") (net 6))
+  (segment (start 105.3764 111.4741) (end 105.3764 107.744) (width 0.25) (layer "B.Cu") (net 6))
+  (segment (start 106.527 113.8) (end 106.527 112.6247) (width 0.25) (layer "B.Cu") (net 6))
+  (segment (start 106.061 107.0594) (end 109.5116 107.0594) (width 0.25) (layer "B.Cu") (net 6))
+  (segment (start 105.3764 107.744) (end 106.061 107.0594) (width 0.25) (layer "B.Cu") (net 6))
   (zone (net 2) (net_name "Earth") (layers F&B.Cu) (hatch edge 0.508)
     (connect_pads (clearance 0.508))
     (min_thickness 0.254) (filled_areas_thickness no)
-    (fill (thermal_gap 0.508) (thermal_bridge_width 0.508))
+    (fill yes (thermal_gap 0.508) (thermal_bridge_width 0.508))
     (polygon
       (pts
         (xy 116.332 116.332)
-        (xy 99.568 116.332)
-        (xy 99.568 99.568)
+        (xy 99.06 116.332)
+        (xy 99.06 99.568)
         (xy 116.332 99.568)
       )

Commit message: single gerber
Routing:
- net Net-(C4-Pad1): track 33.2 -> 33.8 mm
Changed lines of the file:
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@@
     (fp_line (start 1.75 -1.4) (end -1.05 -1.4) (layer "F.Fab") (width 0.1))
     (fp_line (start 1.75 1.4) (end 1.75 -1.4) (layer "F.Fab") (width 0.1))
-    (pad "1" smd roundrect (at -1.625 0 90) (size 1.5 2.35) (layers "F.Cu" "F.Paste" "F.Mask") (roundrect_rratio 0.166667)
+    (pad "1" smd roundrect (at -1.625 0 90) (size 1.5 2.35) (layers "F.Cu" "F.Paste" "F.Mask") (roundrect_rratio 0.1666673333)
       (net 6 "Net-(C4-Pad1)") (pintype "passive"))
-    (pad "2" smd roundrect (at 1.625 0 90) (size 1.5 2.35) (layers "F.Cu" "F.Paste" "F.Mask") (roundrect_rratio 0.166667)
+    (pad "2" smd roundrect (at 1.625 0 90) (size 1.5 2.35) (layers "F.Cu" "F.Paste" "F.Mask") (roundrect_rratio 0.1666673333)
       (net 2 "Earth") (pintype "passive"))
     (model "${KICAD6_3DMODEL_DIR}/Capacitor_Tantalum_SMD.3dshapes/CP_EIA-3528-21_Kemet-B.wrl"
@@
     (fp_line (start -1.75 1.4) (end 1.75 1.4) (layer "F.Fab") (width 0.1))
     (fp_line (start -1.05 -1.4) (end -1.75 -0.7) (layer "F.Fab") (width 0.1))
-    (pad "1" smd roundrect (at -1.625 0 90) (size 1.5 2.35) (layers "F.Cu" "F.Paste" "F.Mask") (roundrect_rratio 0.166667)
+    (pad "1" smd roundrect (at -1.625 0 90) (size 1.5 2.35) (layers "F.Cu" "F.Paste" "F.Mask") (roundrect_rratio 0.1666673333)
       (net 1 "Net-(C1-Pad1)") (pintype "passive"))
-    (pad "2" smd roundrect (at 1.625 0 90) (size 1.5 2.35) (layers "F.Cu" "F.Paste" "F.Mask") (roundrect_rratio 0.166667)
+    (pad "2" smd roundrect (at 1.625 0 90) (size 1.5 2.35) (layers "F.Cu" "F.Paste" "F.Mask") (roundrect_rratio 0.1666673333)
       (net 2 "Earth") (pintype "passive"))
     (model "${KICAD6_3DMODEL_DIR}/Capacitor_Tantalum_SMD.3dshapes/CP_EIA-3528-21_Kemet-B.wrl"
@@
   (segment (start 107.8122 110.6953) (end 107.7744 110.6953) (width 0.2502) (layer "F.Cu") (net 1))
   (segment (start 107.7744 110.6953) (end 107.7366 110.6575) (width 0.5) (layer "F.Cu") (net 1))
-  (via (at 106.104 108.0446) (size 0.8) (drill 0.4) (layers "F.Cu" "B.Cu") (net 1))
+  (via (at 105.8 108.0446) (size 0.8) (drill 0.4) (layers "F.Cu" "B.Cu") (net 1))
   (segment (start 111.607 113.8) (end 111.607 111.019) (width 0.5) (layer "B.Cu") (net 1))
   (segment (start 111.607 111.019) (end 108.6326 108.0446) (width 0.5) (layer "B.Cu") (net 1))
@@
   (segment (start 108.55 109.22) (end 108.55 111.9827) (width 0.5) (layer "B.Cu") (net 2))
   (segment (start 107.85 109.22) (end 108.55 109.22) (width 0.5) (layer "B.Cu") (net 2))
-  (segment (start 106.225 106.1993) (end 106.3657 106.1993) (width 0.25) (layer "F.Cu") (net 3))
+  (segment (start 106.225 103.124) (end 106.225 106.0586) (width 0.25) (layer "F.Cu") (net 3))
+  (segment (start 106.225 106.0586) (end 107.35 107.1836) (width 0.25) (layer "F.Cu") (net 3))
   (segment (start 107.35 107.1836) (end 107.35 107.7825) (width 0.25) (layer "F.Cu") (net 3))
-  (segment (start 106.225 103.124) (end 106.225 106.1993) (width 0.25) (layer "F.Cu") (net 3))
-  (segment (start 106.3657 106.1993) (end 107.35 107.1836) (width 0.25) (layer "F.Cu") (net 3))
   (segment (start 103.987 113.8) (end 106.85 110.937) (width 0.25) (layer "F.Cu") (net 4))
   (segment (start 106.85 110.937) (end 106.85 110.6575) (width 0.25) (layer "F.Cu") (net 4))
-  (segment (start 109.475 103.124) (end 109.475 106.1993) (width 0.25) (layer "F.Cu") (net 5))
-  (segment (start 109.475 106.1993) (end 109.3343 106.1993) (width 0.25) (layer "F.Cu") (net 5))
+  (segment (start 109.475 106.0586) (end 108.35 107.1836) (width 0.25) (layer "F.Cu") (net 5))
+  (segment (start 109.475 103.124) (end 109.475 106.0586) (width 0.25) (layer "F.Cu") (net 5))
   (segment (start 108.35 107.1836) (end 108.35 107.7825) (width 0.25) (layer "F.Cu") (net 5))
-  (segment (start 109.3343 106.1993) (end 108.35 107.1836) (width 0.25) (layer "F.Cu") (net 5))
   (segment (start 113.284 105.765) (end 113.284 107.6745) (width 0.25) (layer "F.Cu") (net 6))
   (segment (start 110.344 107.7825) (end 109.5116 107.7825) (width 0.25) (layer "F.Cu") (net 6))
@@
   (via (at 109.5116 107.0594) (size 0.8) (drill 0.4) (layers "F.Cu" "B.Cu") (net 6))
   (segment (start 106.527 112.6247) (end 105.3764 111.4741) (width 0.25) (layer "B.Cu") (net 6))
-  (segment (start 105.3764 111.4741) (end 105.3764 107.744) (width 0.25) (layer "B.Cu") (net 6))
+  (segment (start 105.555424 107.0594) (end 109.5116 107.0594) (width 0.25) (layer "B.Cu") (net 6))
+  (segment (start 105.075 108.344905) (end 105.075 107.539824) (width 0.25) (layer "B.Cu") (net 6))
+  (segment (start 105.3764 108.646305) (end 105.075 108.344905) (width 0.25) (layer "B.Cu") (net 6))
+  (segment (start 105.075 107.539824) (end 105.555424 107.0594) (width 0.25) (layer "B.Cu") (net 6))
+  (segment (start 105.3764 111.4741) (end 105.3764 108.646305) (width 0.25) (layer "B.Cu") (net 6))
   (segment (start 106.527 113.8) (end 106.527 112.6247) (width 0.25) (layer "B.Cu") (net 6))
-  (segment (start 106.061 107.0594) (end 109.5116 107.0594) (width 0.25) (layer "B.Cu") (net 6))
-  (segment (start 105.3764 107.744) (end 106.061 107.0594) (width 0.25) (layer "B.Cu") (net 6))
   (zone (net 2) (net_name "Earth") (layers F&B.Cu) (hatch edge 0.508)
     (connect_pads (clearance 0.508))
